File: schematics/qtpy_synth_proto2a.brd (EAGLE design)
At the start: 76.2 x 63.5 mm, 26 parts, among them IC1 H11L1MS, J1 AUDIO-JACK-TRRS, J2 AUDIO-JACK-TRRS, P1 10k, P2 10k, U1 ADAFRUIT_QTPYM0

Commit message: fix name, add hwtest
Other:
- board text added: "qtpy_synth_proto2a"
- board text added: "works with CircuitPython!"
Changed lines of the file:
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@@
 <grid distance="0.05" unitdist="inch" unit="inch" style="lines" multiple="1" display="no" altdistance="0.01" altunitdist="inch" altunit="inch"/>
 <layers>
-<layer number="1" name="Top" color="4" fill="1" visible="yes" active="yes"/>
+<layer number="1" name="Top" color="4" fill="1" visible="no" active="yes"/>
 <layer number="2" name="Route2" color="1" fill="3" visible="no" active="no"/>
 <layer number="3" name="Route3" color="4" fill="3" visible="no" active="no"/>
@@
 <text x="70.104" y="49.022" size="1.27" layer="21" ratio="10" rot="R90">AUDIO OUT</text>
 <text x="24.13" y="55.626" size="1.27" layer="21" ratio="10">@todbot</text>
-<text x="72.39" y="46.99" size="1.778" layer="22" ratio="10" rot="MR0">qtpy_synth</text>
-<text x="72.39" y="44.45" size="1.016" layer="22" ratio="10" rot="MR0">github.com/todbot/qtpy_synth</text>
-<text x="72.39" y="41.91" size="1.016" layer="22" ratio="10" rot="MR0">27 Jun 2023 - @todbot </text>
-<text x="72.39" y="38.1" size="1.016" layer="22" ratio="10" rot="MR0" align="top-left">Parts:
+<text x="72.39" y="39.37" size="1.778" layer="22" ratio="10" rot="MR0">qtpy_synth</text>
+<text x="72.39" y="36.83" size="1.016" layer="22" ratio="10" rot="MR0">github.com/todbot/qtpy_synth</text>
+<text x="72.39" y="31.75" size="1.016" layer="22" ratio="10" rot="MR0">27 Jun 2023 - @todbot </text>
+<text x="68.58" y="11.43" size="1.016" layer="22" ratio="10" rot="MR0" align="top-left">Parts:
 - QTPy RP2040
 - 0.9" I2C OLED SSD1306
@@
 SCL
 SW</text>
+<text x="19.05" y="-1.27" size="1.016" layer="22" ratio="10" rot="MR0">qtpy_synth_proto2a</text>
+<text x="72.39" y="34.29" size="1.016" layer="22" ratio="10" rot="MR0">works with CircuitPython!</text>
 </plain>
 <attributes>
