File: schematics/qtpy_synth_proto2b.brd (EAGLE design)
At the start: 76.2 x 63.5 mm, 25 parts, among them IC1 H11L1MS, J1 AUDIO-JACK-TRRS, J2 AUDIO-JACK-TRRS, P1 10k, P2 10k, U1 ADAFRUIT_QTPYM0

Commit message: cleanup proto2b pcb before fab submit
Routing:
- net MIDI_IN: track 37.4 -> 39.0 mm
- net POTA: track 44.2 -> 44.9 mm
Other:
- board text added: "12 Jul 2023 - @todbot"
- board text added: "5V GND 3V AUDIO TP3 TP4 MIDI"
- board text added: "AUDIO LINE OUT"
- board text added: "Parts: - QTPy RP2040 - 0.9" I2C OLED SSD1306 - 2x 10k pots - tact switch 6mm - 2x PJ320D 3.5mm jacks - IC1: H11L1 optoisolator - D1: 1N4148 - R1-R4: 1M, R5: 4.7k, R6,R7: 220, R8: 100: R9: 1.8k - C1,C2: 100nF, C3: 47uF"
- board text removed: "27 Jun 2023 - @todbot"
- board text removed: "5V GND 3V PWM TP3 TP4 MIDI"
- board text removed: "Parts: - QTPy RP2040 - 0.9" I2C OLED SSD1306 - 2x 10k pots - tact switch - 2x PJ320D 3.5mm jacks - IC1: H11L1 optoisolator - D1: 1N4148 - R1-4: 1M, R5: 4.7k, R6,R7: 220, R8:100: R9 1.8k - C1,C2: 100nF, C3: 47uF"
